File: RP2040_base.kicad_sch (KiCad schematic)
At the start: 24 parts, among them J2 Conn_01x02, U1 W25Q16JV, U2 RP2040, Y2 ECS-120-8-33-JGN-TR3

Commit message: Add git url
Connections:
- no-connect marks 0 -> 1
Other:
- company: (none) -> https://github.com/TT-392/RP2040-base
Changed lines of the file:
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@@
     (date "2023-07-22")
     (rev "0.1")
+    (company "https://github.com/TT-392/RP2040-base")
   )
   (junction (at 88.9 147.32) (diameter 0) (color 0 0 0 0)
@@
   (junction (at 255.27 31.75) (diameter 0) (color 0 0 0 0)
   )
+  (no_connect (at 170.18 151.13))
   (wire (pts (xy 95.25 147.32) (xy 105.41 147.32))
     (stroke (width 0) (type default))

Commit message: Create sample pcb layout, manage schematic files better, and fill in missing 3d model.
Parts:
- removed J2: Conn_01x02, Connector_PinHeader_2.54mm:PinHeader_1x02_P2.54mm_Horizontal, symbol Connector_Generic:Conn_01x02
- removed R9: DNF, Resistor_SMD:R_0603_1608Metric, symbol Device:R
- added C9: 100n, Capacitor_SMD:C_0402_1005Metric, symbol Device:C
- added SW1: SW_Push, RP2040_base:TS-1187A, symbol Switch:SW_Push
- U1: footprint Package_SO:SOIC-8_5.23x5.23mm_P1.27mm -> SOIC-8_5.275x5.275mm_P1.27mm
Connections:
- net GND: now also C9.2, SW1.1
- net VIN: now also C9.1
- net ~{USB_BOOT}: now also SW1.2
Changed lines of the file:
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@@
   (title_block
     (title "RP2040 Base")
-    (date "2023-07-22")
-    (rev "0.1")
+    (date "2023-07-25")
+    (rev "0.2")
     (company "https://github.com/TT-392/RP2040-base")
   )
-  (junction (at 88.9 147.32) (diameter 0) (color 0 0 0 0)
-  )
   (junction (at 189.23 46.99) (diameter 0) (color 0 0 0 0)
   )
@@
   (junction (at 255.27 43.18) (diameter 0) (color 0 0 0 0)
   )
+  (junction (at 278.13 43.18) (diameter 0) (color 0 0 0 0)
+  )
   (junction (at 67.31 105.41) (diameter 0) (color 0 0 0 0)
   )
@@
   (junction (at 198.12 31.75) (diameter 0) (color 0 0 0 0)
   )
-  (junction (at 76.2 163.83) (diameter 0) (color 0 0 0 0)
+  (junction (at 266.7 31.75) (diameter 0) (color 0 0 0 0)
   )
   (junction (at 243.84 43.18) (diameter 0) (color 0 0 0 0)
@@
     (stroke (width 0) (type default))
   )
-  (wire (pts (xy 41.91 166.37) (xy 43.18 166.37))
-    (stroke (width 0) (type default))
-  )
   (wire (pts (xy 134.62 82.55) (xy 128.27 82.55))
     (stroke (width 0) (type default))
@@
     (stroke (width 0) (type default))
   )
-  (wire (pts (xy 76.2 148.59) (xy 76.2 147.32))
+  (wire (pts (xy 30.48 163.83) (xy 31.75 163.83))
     (stroke (width 0) (type default))
   )
@@
     (stroke (width 0) (type default))
   )
-  (wire (pts (xy 266.7 43.18) (xy 266.7 44.45))
+  (wire (pts (xy 278.13 43.18) (xy 278.13 44.45))
     (stroke (width 0) (type default))
   )
@@
     (stroke (width 0) (type default))
   )
+  (wire (pts (xy 278.13 43.18) (xy 278.13 40.64))
+    (stroke (width 0) (type default))
+  )
   (wire (pts (xy 189.23 31.75) (xy 189.23 46.99))
     (stroke (width 0) (type default))
   )
+  (wire (pts (xy 266.7 43.18) (xy 278.13 43.18))
+    (stroke (width 0) (type default))
+  )
   (wire (pts (xy 176.53 64.77) (xy 176.53 62.23))
     (stroke (width 0) (type default))
@@
     (stroke (width 0) (type default))
   )
-  (wire (pts (xy 76.2 147.32) (xy 88.9 147.32))
-    (stroke (width 0) (type default))
-  )
   (wire (pts (xy 209.55 31.75) (xy 220.98 31.75))
     (stroke (width 0) (type default))
@@
     (stroke (width 0) (type default))
   )
+  (wire (pts (xy 278.13 31.75) (xy 266.7 31.75))
+    (stroke (width 0) (type default))
+  )
   (wire (pts (xy 67.31 115.57) (xy 81.28 115.57))
     (stroke (width 0) (type default))
   )
-  (wire (pts (xy 76.2 163.83) (xy 78.74 163.83))
+  (wire (pts (xy 62.23 163.83) (xy 78.74 163.83))
     (stroke (width 0) (type default))
   )
@@
     (stroke (width 0) (type default))
   )
-  (wire (pts (xy 62.23 163.83) (xy 76.2 163.83))
-    (stroke (width 0) (type default))
-  )
   (wire (pts (xy 78.74 168.91) (xy 64.77 168.91))
     (stroke (width 0) (type default))
@@
     (stroke (width 0) (type default))
   )
-  (wire (pts (xy 43.18 166.37) (xy 43.18 167.64))
-    (stroke (width 0) (type default))
-  )
   (wire (pts (xy 95.25 148.59) (xy 95.25 147.32))
     (stroke (width 0) (type default))
@@
     (stroke (width 0) (type default))
   )
+  (wire (pts (xy 278.13 33.02) (xy 278.13 31.75))
+    (stroke (width 0) (type default))
+  )
   (wire (pts (xy 153.67 105.41) (xy 139.7 105.41))
     (stroke (width 0) (type default))
@@
     (stroke (width 0) (type default))
   )
-  (wire (pts (xy 76.2 156.21) (xy 76.2 163.83))
-    (stroke (width 0) (type default))
+  (text_box "USB Differential pair impedance should be 90 ohms, spacing differential pair traces should be 1.275mm, here is a table for trace thickness because I was lazy, and used an online calculator. USB isn't really that crytical in practice though, so I ended up using 1mm on the 1.6mm 2 layer pcb\n\nHorizontal spacing	track width\n1.51				1.138\n1.3					0.997\n1.2					0.93\n1.1					0.863\n1					0.795\n0.5					0.454\n0.2					0.229\n0.1					0.128\n"
+    (at 62.23 34.29 0) (size 41.91 38.1)
+    (stroke (width 0) (type default))
+    (fill (type none))
+    (effects (font (size 1.27 1.27)) (justify left top))
   )
   (text "Flash" (at 46.99 148.59 0)
@@
     (effects (font (size 1.27 1.27)) (justify left bottom))
   )
-  (label "GND" (at 266.7 44.45 270) (fields_autoplaced)
+  (label "GND" (at 278.13 44.45 270) (fields_autoplaced)
     (effects (font (size 1.27 1.27)) (justify right bottom))
   )
@@
     (effects (font (size 1.27 1.27)) (justify left bottom))
   )
-  (label "GND" (at 43.18 167.64 270) (fields_autoplaced)
+  (label "GND" (at 30.48 163.83 270) (fields_autoplaced)
     (effects (font (size 1.27 1.27)) (justify right bottom))
   )
@@
     (effects (font (size 1.27 1.27)) (justify left))
   )
+  (symbol (lib_id "Device:C") (at 278.13 36.83 0) (unit 1)
+    (in_bom yes) (on_board yes) (dnp no)
+    (property "Reference" "C9" (at 281.051 35.6616 0)
+      (effects (font (size 1.27 1.27)) (justify left))
+    )
+    (property "Value" "100n" (at 281.051 37.973 0)
+      (effects (font (size 1.27 1.27)) (justify left))
+    )
+    (property "Footprint" "Capacitor_SMD:C_0402_1005Metric" (at 279.0952 40.64 0)
+      (effects (font (size 1.27 1.27)) hide)
+    )
+    (property "Datasheet" "~" (at 278.13 36.83 0)
+      (effects (font (size 1.27 1.27)) hide)
+    )
+    (property "Pin" "49" (at 275.59 39.37 0)
+      (effects (font (size 1.27 1.27)))
+    )
+    (pin "1")
+    (pin "2")
+    (instances
+      (project "RP2040_base"
+        (path "/bff3622d-c437-4efa-a243-896582301865"
+          (reference "C9") (unit 1)
+        )
+      )
+      (project "arisu"
+        (path "/fd2aa641-4342-4b9c-83bf-54ed9335b528/769dae23-5223-4917-97f1-926f10044dd4"
+          (reference "C34") (unit 1)
+        )
+      )
+    )
+  )
   (symbol (lib_id "Device:R") (at 85.09 115.57 270) (unit 1)
     (in_bom yes) (on_board yes) (dnp no)
@@
         (path "/fd2aa641-4342-4b9c-83bf-54ed9335b528/769dae23-5223-4917-97f1-926f10044dd4"
           (reference "C36") (unit 1)
-        )
-      )
-    )
-  )
-  (symbol (lib_id "Device:R") (at 76.2 152.4 0) (unit 1)
-    (in_bom yes) (on_board yes) (dnp no)
-    (property "Reference" "R9" (at 77.978 151.2316 0)
-      (effects (font (size 1.27 1.27)) (justify left))
-    )
-    (property "Value" "DNF" (at 77.978 153.543 0)
-      (effects (font (size 1.27 1.27)) (justify left))
-    )
-    (property "Footprint" "Resistor_SMD:R_0603_1608Metric" (at 74.422 152.4 90)
-      (effects (font (size 1.27 1.27)) hide)
-    )
-    (property "Datasheet" "~" (at 76.2 152.4 0)
-      (effects (font (size 1.27 1.27)) hide)
-    )
-    (pin "1")
-    (pin "2")
-    (instances
-      (project "RP2040_base"
-        (path "/bff3622d-c437-4efa-a243-896582301865"
-          (reference "R9") (unit 1)
-        )
-      )
-      (project "arisu"
-        (path "/fd2aa641-4342-4b9c-83bf-54ed9335b528/769dae23-5223-4917-97f1-926f10044dd4"
-          (reference "R14") (unit 1)
         )
       )
@@
       (effects (font (size 1.27 1.27)) (justify left))
     )
-    (property "Footprint" "Package_SO:SOIC-8_5.23x5.23mm_P1.27mm" (at 88.9 171.45 0)
+    (property "Footprint" "SOIC-8_5.275x5.275mm_P1.27mm" (at 88.9 171.45 0)
       (effects (font (size 1.27 1.27)) hide)
     )
     (property "Datasheet" "" (at 88.9 171.45 0)
+      (effects (font (size 1.27 1.27)) hide)
+    )
+    (property "GIT_URL" "" (at 88.9 171.45 0)
+      (effects (font (size 1.27 1.27)))
+    )
+    (property "Untitled Field" "" (at 88.9 171.45 0)
       (effects (font (size 1.27 1.27)) hide)
     )
@@
     )
   )
-  (symbol (lib_id "Connector_Generic:Conn_01x02") (at 36.83 163.83 0) (mirror y) (unit 1)
-    (in_bom yes) (on_board yes) (dnp no)
-    (property "Reference" "J2" (at 35.56 160.02 0)
-      (effects (font (size 1.27 1.27)))
-    )
-    (property "Value" "Conn_01x02" (at 35.56 170.18 0)
-      (effects (font (size 1.27 1.27)))
-    )
-    (property "Footprint" "Connector_PinHeader_2.54mm:PinHeader_1x02_P2.54mm_Horizontal" (at 36.83 163.83 0)
-      (effects (font (size 1.27 1.27)) hide)
-    )
-    (property "Datasheet" "~" (at 36.83 163.83 0)
-      (effects (font (size 1.27 1.27)) hide)
-    )
-    (pin "1")
-    (pin "2")
-    (instances
-      (project "RP2040_base"
-        (path "/bff3622d-c437-4efa-a243-896582301865"
-          (reference "J2") (unit 1)
-        )
-      )
-      (project "arisu"
-        (path "/fd2aa641-4342-4b9c-83bf-54ed9335b528/769dae23-5223-4917-97f1-926f10044dd4"
-          (reference "J5") (unit 1)
-        )
-      )
-    )
-  )
   (symbol (lib_id "Device:C") (at 52.07 115.57 270) (unit 1)
     (in_bom yes) (on_board yes) (dnp no)
@@
         )
       )
+    )
+  )
+  (symbol (lib_id "Switch:SW_Push") (at 36.83 163.83 0) (unit 1)
+    (in_bom yes) (on_board yes) (dnp no) (fields_autoplaced)
+    (property "Reference" "SW1" (at 36.83 157.8991 0)
+      (effects (font (size 1.27 1.27)))
+    )
+    (property "Value" "SW_Push" (at 36.83 159.8201 0)
+      (effects (font (size 1.27 1.27)))
+    )
+    (property "Footprint" "RP2040_base:TS-1187A" (at 36.83 158.75 0)
+      (effects (font (size 1.27 1.27)) hide)
+    )
+    (property "Datasheet" "~" (at 36.83 158.75 0)
+      (effects (font (size 1.27 1.27)) hide)
+    )
+    (property "GIT_URL" "" (at 36.83 163.83 0)
+      (effects (font (size 1.27 1.27)))
+    )
+    (property "Untitled Field" "" (at 36.83 163.83 0)
+      (effects (font (size 1.27 1.27)) hide)
+    )
+    (pin "1")
+    (pin "2")
+    (instances
+      (project "RP2040_base"
+        (path "/bff3622d-c437-4efa-a243-896582301865"
+          (reference "SW1") (unit 1)
+        )
+      )
