File: RP2040_base_example.kicad_sch (KiCad schematic)
At the start: 10 parts, among them J1 Conn_01x17, J2 Conn_01x17, J4 USB_C_Receptacle_USB2.0, U3 AMS1117-3.3

Commit message: Reannotate
Parts:
- J1, J2: footprint (none) -> Connector_PinHeader_1.27mm:PinHeader_1x17_P1.27mm_Vertical
- R5: renamed from R3; footprint (none) -> Resistor_SMD:R_0603_1608Metric
- SWD1: renamed from SWD; footprint (none) -> Connector_PinHeader_1.27mm:PinHeader_1x03_P1.27mm_Vertical
- renumbered J4 to J3, R1 to R6, R2 to R7
