File: RP2040_base_example.kicad_sch (KiCad schematic)
At the start: 10 parts, among them J1 Conn_01x03, J2 Conn_01x13, J3 GT-USB-7047C, U1 XC6206P332MR, U2 SRV05-4

Commit message: Rotate footprints to coincide with jlcpcb rotation
Parts:
- U1: footprint Package_TO_SOT_SMD:SOT-23-3 -> footprints:SOT-23-3_flipped_for_jlcpcb
- U2: footprint Package_TO_SOT_SMD:SOT-23-6 -> footprints:SOT-23-6_flipped_for_jlcpcb
Changed lines of the file:
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@@
       (effects (font (size 1.27 1.27)) (justify left))
     )
-    (property "Footprint" "Package_TO_SOT_SMD:SOT-23-6" (at 99.06 140.97 0)
+    (property "Footprint" "footprints:SOT-23-6_flipped_for_jlcpcb" (at 99.06 140.97 0)
       (effects (font (size 1.27 1.27)) hide)
     )
@@
     )
     (property "LCSC" "C85364" (at 84.4297 116.3701 0)
+      (effects (font (size 1.27 1.27)) hide)
+    )
+    (property "GIT_URL" "" (at 81.28 129.54 0)
+      (effects (font (size 1.27 1.27)))
+    )
+    (property "Untitled Field" "" (at 81.28 129.54 0)
       (effects (font (size 1.27 1.27)) hide)
     )
@@
       (effects (font (size 1.27 1.27)))
     )
-    (property "Footprint" "Package_TO_SOT_SMD:SOT-23-3" (at 93.98 31.115 0)
+    (property "Footprint" "footprints:SOT-23-3_flipped_for_jlcpcb" (at 93.98 31.115 0)
       (effects (font (size 1.27 1.27) italic) hide)
     )
@@
       (effects (font (size 1.27 1.27)) hide)
     )
+    (property "GIT_URL" "" (at 93.98 36.83 0)
+      (effects (font (size 1.27 1.27)))
+    )
+    (property "Untitled Field" "" (at 93.98 36.83 0)
+      (effects (font (size 1.27 1.27)) hide)
+    )

Commit message: Add title blocks, and set version to 0.9 (will bump to 1.0 if ordered and tested)
Other:
- company: (none) -> https://github.com/TT-392/RP2040-base-example
- title: (none) -> RP2040-base example
Changed lines of the file:
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@@
 (kicad_sch (version 20230121) (generator eeschema)
   (paper "A4")
+  (title_block
+    (title "RP2040-base example")
+    (date "2023-07-30")
+    (rev "0.9")
+    (company "https://github.com/TT-392/RP2040-base-example")
+  )
   (junction (at 49.53 106.68) (diameter 0) (color 0 0 0 0)
   )
